Commit message: tunnelling in pybullet working

File: terrain/bauzil_stairs.urdf (robot description, URDF)
Before this commit: robot bauzil_stairs.urdf, 1 links, 0 joints
Links:
- link baseLink: geometry collision mesh filename=Block.stl scale=0.0015 0.0005 0.00075; collision mesh filename=Block.stl scale=0.0015 0.0005 0.00075
